Commit message: Port reviewed Wonik QD simulation to ROS 2 Humble

File: wonik_cobot_v2_description/urdf/wonik_cobot_v2.gazebo.xacro (robot description, xacro)
@@ -68,48 +68,49 @@
             </clip>
           </camera>
-          <plugin name="depth_camera_controller" filename="libgazebo_ros_openni_kinect.so">
-            <alwaysOn>true</alwaysOn>
-            <updateRate>15</updateRate>
-            <cameraName>camera</cameraName>
-            <imageTopicName>rgb/image_raw</imageTopicName>
-            <cameraInfoTopicName>rgb/camera_info</cameraInfoTopicName>
-            <depthImageTopicName>depth/image_raw</depthImageTopicName>
-            <depthImageCameraInfoTopicName>depth/camera_info</depthImageCameraInfoTopicName>
-            <pointCloudTopicName>depth/points</pointCloudTopicName>
-            <frameName>camera_depth_optical_frame</frameName>
-            <pointCloudCutoff>0.1</pointCloudCutoff>
-            <pointCloudCutoffMax>6.0</pointCloudCutoffMax>
-            <baseline>0.05</baseline>
-            <distortionK1>0</distortionK1>
-            <distortionK2>0</distortionK2>
-            <distortionK3>0</distortionK3>
-            <distortionT1>0</distortionT1>
-            <distortionT2>0</distortionT2>
-            <CxPrime>0</CxPrime>
-            <Cx>0</Cx>
-            <Cy>0</Cy>
-            <focalLength>0</focalLength>
-            <hackBaseline>0</hackBaseline>
+          <plugin name="depth_camera_controller" filename="libgazebo_ros_camera.so">
+            <ros>
+              <namespace>/camera</namespace>
+              <remapping>camera/points:=depth/points</remapping>
+              <remapping>camera/image_raw:=rgb/image_raw</remapping>
+              <remapping>camera/camera_info:=rgb/camera_info</remapping>
+              <remapping>camera/depth/image_raw:=depth/image_raw</remapping>
+              <remapping>camera/depth/camera_info:=depth/camera_info</remapping>
+            </ros>
+            <camera_name>camera</camera_name><frame_name>camera_depth_optical_frame</frame_name>
+            <min_depth>0.1</min_depth><max_depth>6.0</max_depth>
           </plugin>
         </sensor>
       </gazebo>
     </xacro:if>
+    <!-- IMU: /imu/data (frame imu_link) at 200 Hz. The noise is a typical MEMS gyro (0.005 rad/s) and
+         also sets the message covariances (noise^2). No bias: robot_localization does not estimate one,
+         so a real gyro needs its bias removed by the driver (e.g. calibrated at standstill). -->
+    <gazebo reference="imu_link">
+      <sensor name="imu_sensor" type="imu">
+        <always_on>true</always_on>
+        <update_rate>200</update_rate>
+        <imu>
+          <angular_velocity>
+            <x><noise type="gaussian"><mean>0</mean><stddev>0.005</stddev></noise></x>
+            <y><noise type="gaussian"><mean>0</mean><stddev>0.005</stddev></noise></y>
+            <z><noise type="gaussian"><mean>0</mean><stddev>0.005</stddev></noise></z>
+          </angular_velocity>
+        </imu>
+        <plugin name="imu_plugin" filename="libgazebo_ros_imu_sensor.so">
+          <ros><remapping>~/out:=/imu/data</remapping></ros>
+          <frame_name>imu_link</frame_name><initial_orientation_as_reference>false</initial_orientation_as_reference>
+        </plugin>
+      </sensor>
+    </gazebo>
     <gazebo>
       <!-- Steer joints: position, drive joints: velocity (as on the real drive units). -->
-      <plugin name="gazebo_ros_control" filename="libgazebo_ros_control.so">
-        <robotNamespace>/</robotNamespace>
-        <robotSimType>gazebo_ros_control/DefaultRobotHWSim</robotSimType>
-        <legacyModeNS>true</legacyModeNS>
+      <plugin name="gazebo_ros2_control" filename="libgazebo_ros2_control.so">
+        <parameters>$(find wonik_cobot_v2_bringup)/config/controllers.yaml</parameters>
       </plugin>
       <!-- Ground truth of base_footprint for evaluation: /ground_truth/odom in frame world, no TF. -->
       <plugin name="ground_truth" filename="libgazebo_ros_p3d.so">
-        <alwaysOn>true</alwaysOn>
-        <updateRate>50.0</updateRate>
-        <bodyName>base_footprint</bodyName>
-        <topicName>ground_truth/odom</topicName>
-        <frameName>world</frameName>
-        <gaussianNoise>0.0</gaussianNoise>
-        <xyzOffsets>0 0 0</xyzOffsets>
-        <rpyOffsets>0 0 0</rpyOffsets>
+        <ros><remapping>odom:=/ground_truth/odom</remapping></ros>
+        <update_rate>50.0</update_rate><body_name>base_footprint</body_name>
+        <frame_name>world</frame_name><gaussian_noise>0.0</gaussian_noise>
       </plugin>
       <xacro:if value="${kinematic}">

File: wonik_cobot_v2_description/urdf/wonik_cobot_v2.urdf.xacro (robot description, xacro)
@@ -10,5 +10,4 @@
   <!-- Gazebo depth camera sensor; it needs an X display (rendering) to produce images -->
   <xacro:arg name="depth_camera" default="true"/>
-  <xacro:include filename="$(find velodyne_description)/urdf/HDL-32E.urdf.xacro"/>
   <xacro:include filename="$(find wonik_cobot_v2_description)/urdf/wonik_cobot_v2.gazebo.xacro"/>
   <xacro:property name="g" value="${xacro.load_yaml('$(arg geometry)')}"/>
@@ -88,22 +87,4 @@
       </collision>
     </link>
-    <transmission name="${name}_steer_trans">
-      <type>transmission_interface/SimpleTransmission</type>
-      <joint name="${name}_steer_joint">
-        <hardwareInterface>hardware_interface/PositionJointInterface</hardwareInterface>
-      </joint>
-      <actuator name="${name}_steer_motor">
-        <mechanicalReduction>1</mechanicalReduction>
-      </actuator>
-    </transmission>
-    <transmission name="${name}_drive_trans">
-      <type>transmission_interface/SimpleTransmission</type>
-      <joint name="${name}_drive_joint">
-        <hardwareInterface>hardware_interface/VelocityJointInterface</hardwareInterface>
-      </joint>
-      <actuator name="${name}_drive_motor">
-        <mechanicalReduction>1</mechanicalReduction>
-      </actuator>
-    </transmission>
   </xacro:macro>
   <!-- Passive omni wheel: sphere contact (its visual is part of base.stl). -->
@@ -140,9 +121,31 @@
   <xacro:qd_units/>
   <xacro:omni_wheels/>
-  <!-- 3D LiDAR (velodyne_simulator), stand-in for the Mid-360. Topic /points, frame velodyne. -->
+  <!-- 3D LiDAR (velodyne_simulator), stand-in for the Mid-360. Topic /points, frame velodyne.
+       min_range 0.3 m instead of the HDL-32E's 0.9 m, closer to the Mid-360 (0.1 m): obstacles right
+       beside the body must be visible (turn-in-place check); 0.3 m keeps most deck hits out. -->
   <xacro:property name="l" value="${g['lidar_xyz']}"/>
-  <xacro:HDL-32E parent="base_link" name="velodyne" topic="/points" hz="10" samples="625" gpu="$(arg lidar_gpu)">
-    <origin xyz="${l[0]} ${l[1]} ${l[2]}" rpy="0 0 0"/>
-  </xacro:HDL-32E>
+  <link name="velodyne">
+    <inertial><mass value="0.8"/><inertia ixx="0.001" ixy="0" ixz="0" iyy="0.001" iyz="0" izz="0.001"/></inertial>
+    <visual><geometry><cylinder radius="0.04" length="0.07"/></geometry></visual>
+  </link>
+  <joint name="velodyne_joint" type="fixed">
+    <parent link="base_link"/><child link="velodyne"/><origin xyz="${l[0]} ${l[1]} ${l[2]}" rpy="0 0 0"/>
+  </joint>
+  <gazebo reference="velodyne">
+    <sensor name="lidar" type="${'gpu_ray' if '$(arg lidar_gpu)' == 'true' else 'ray'}">
+      <always_on>true</always_on><update_rate>10</update_rate>
+      <ray>
+        <scan>
+          <horizontal><samples>625</samples><resolution>1</resolution><min_angle>-3.14159265</min_angle><max_angle>3.14159265</max_angle></horizontal>
+          <vertical><samples>32</samples><resolution>1</resolution><min_angle>-0.5353</min_angle><max_angle>0.1862</max_angle></vertical>
+        </scan>
+        <range><min>0.3</min><max>30.0</max><resolution>0.01</resolution></range>
+      </ray>
+      <plugin name="lidar_ros" filename="libgazebo_ros_ray_sensor.so">
+        <ros><remapping>~/out:=/points</remapping></ros>
+        <output_type>sensor_msgs/PointCloud2</output_type><frame_name>velodyne</frame_name>
+      </plugin>
+    </sensor>
+  </gazebo>
   <!-- Front depth camera (RealSense D435). camera_depth_optical_frame: z forward, x right, y down. -->
   <xacro:property name="c" value="${g['depth_camera_xyz']}"/>
@@ -170,4 +173,38 @@
   </joint>
   <link name="camera_depth_optical_frame"/>
+  <!-- IMU: /imu/data in frame imu_link -->
+  <xacro:property name="i" value="${g['imu_xyz']}"/>
+  <xacro:property name="ir" value="${g['imu_rpy']}"/>
+  <joint name="imu_joint" type="fixed">
+    <origin xyz="${i[0]} ${i[1]} ${i[2]}" rpy="${ir[0]} ${ir[1]} ${ir[2]}"/>
+    <parent link="base_link"/>
+    <child link="imu_link"/>
+  </joint>
+  <link name="imu_link">
+    <inertial>
+      <mass value="0.01"/>
+      <origin xyz="0 0 0"/>
+      <inertia ixx="1e-6" ixy="0" ixz="0" iyy="1e-6" iyz="0" izz="1e-6"/>
+    </inertial>
+  </link>
   <xacro:cobot_v2_gazebo sim_drive="$(arg sim_drive)" depth_camera="$(arg depth_camera)"/>
+  <xacro:arg name="hardware_plugin" default="gazebo_ros2_control/GazeboSystem"/>
+  <ros2_control name="WonikSystem" type="system">
+    <hardware><plugin>$(arg hardware_plugin)</plugin></hardware>
+    <xacro:macro name="control_modules" params="i:=0">
+      <xacro:if value="${i &lt; len(g['module_names'])}">
+        <joint name="${g['steer_joints'][i]}">
+          <command_interface name="position"/>
+          <state_interface name="position"><param name="initial_value">0.0</param></state_interface>
+          <state_interface name="velocity"/>
+        </joint>
+        <joint name="${g['drive_joints'][i]}">
+          <command_interface name="velocity"/>
+          <state_interface name="position"/><state_interface name="velocity"/>
+        </joint>
+        <xacro:control_modules i="${i+1}"/>
+      </xacro:if>
+    </xacro:macro>
+    <xacro:control_modules/>
+  </ros2_control>
 </robot>
