Commit message: Add the front depth camera (RealSense D435) to cobot_v2
Camera frames at the D435 position in the CAD (front face, 0.24 m high),
looking forward; in Gazebo an openni_kinect depth sensor publishes
/camera/depth/points at 15 Hz with the D435 field of view. The sensor
can be left out with depth_camera:=false (it needs an X display to
render).

Co-Authored-By: Claude Opus 5.5 <noreply@anthropic.com>

File: wonik_cobot_v2_description/urdf/wonik_cobot_v2.gazebo.xacro (robot description, xacro)
@@ -8,5 +8,5 @@
                              brings. For checking the kinematics and wheel odometry. -->
 <robot xmlns:xacro="http://www.ros.org/wiki/xacro">
-  <xacro:macro name="cobot_v2_gazebo" params="sim_drive">
+  <xacro:macro name="cobot_v2_gazebo" params="sim_drive depth_camera:=true">
     <xacro:property name="kinematic" value="${sim_drive == 'kinematic'}"/>
     <xacro:if value="${sim_drive not in ['kinematic', 'physics']}">
@@ -50,4 +50,49 @@
     </xacro:macro>
     <xacro:omni_wheels_gazebo/>
+    <!-- Front depth camera: /camera/depth/points (frame camera_depth_optical_frame), 15 Hz, D435 FOV -->
+    <xacro:if value="${depth_camera}">
+      <gazebo reference="camera_link">
+        <sensor type="depth" name="depth_camera">
+          <always_on>true</always_on>
+          <update_rate>15</update_rate>
+          <camera>
+            <horizontal_fov>1.5184</horizontal_fov>
+            <image>
+              <format>R8G8B8</format>
+              <width>424</width>
+              <height>240</height>
+            </image>
+            <clip>
+              <near>0.1</near>
+              <far>10.0</far>
+            </clip>
+          </camera>
+          <plugin name="depth_camera_controller" filename="libgazebo_ros_openni_kinect.so">
+            <alwaysOn>true</alwaysOn>
+            <updateRate>15</updateRate>
+            <cameraName>camera</cameraName>
+            <imageTopicName>rgb/image_raw</imageTopicName>
+            <cameraInfoTopicName>rgb/camera_info</cameraInfoTopicName>
+            <depthImageTopicName>depth/image_raw</depthImageTopicName>
+            <depthImageCameraInfoTopicName>depth/camera_info</depthImageCameraInfoTopicName>
+            <pointCloudTopicName>depth/points</pointCloudTopicName>
+            <frameName>camera_depth_optical_frame</frameName>
+            <pointCloudCutoff>0.1</pointCloudCutoff>
+            <pointCloudCutoffMax>6.0</pointCloudCutoffMax>
+            <baseline>0.05</baseline>
+            <distortionK1>0</distortionK1>
+            <distortionK2>0</distortionK2>
+            <distortionK3>0</distortionK3>
+            <distortionT1>0</distortionT1>
+            <distortionT2>0</distortionT2>
+            <CxPrime>0</CxPrime>
+            <Cx>0</Cx>
+            <Cy>0</Cy>
+            <focalLength>0</focalLength>
+            <hackBaseline>0</hackBaseline>
+          </plugin>
+        </sensor>
+      </gazebo>
+    </xacro:if>
     <gazebo>
       <!-- Steer joints: position, drive joints: velocity (as on the real drive units). -->

File: wonik_cobot_v2_description/urdf/wonik_cobot_v2.urdf.xacro (robot description, xacro)
@@ -3,9 +3,11 @@
      Meshes are visual only (converted from cobot_v2_asm.stp); collisions are primitives.
      Everything Gazebo-specific is in wonik_cobot_v2.gazebo.xacro (ignored outside Gazebo).
-       xacro wonik_cobot_v2.urdf.xacro [sim_drive:=kinematic|physics] [lidar_gpu:=true] -->
+       xacro wonik_cobot_v2.urdf.xacro [sim_drive:=kinematic|physics] [lidar_gpu:=true] [depth_camera:=false] -->
 <robot name="wonik_cobot_v2" xmlns:xacro="http://www.ros.org/wiki/xacro">
   <xacro:arg name="geometry" default="$(find wonik_cobot_v2_description)/config/geometry.yaml"/>
   <xacro:arg name="sim_drive" default="kinematic"/>
   <xacro:arg name="lidar_gpu" default="false"/>
+  <!-- Gazebo depth camera sensor; it needs an X display (rendering) to produce images -->
+  <xacro:arg name="depth_camera" default="true"/>
   <xacro:include filename="$(find velodyne_description)/urdf/HDL-32E.urdf.xacro"/>
   <xacro:include filename="$(find wonik_cobot_v2_description)/urdf/wonik_cobot_v2.gazebo.xacro"/>
@@ -143,4 +145,29 @@
     <origin xyz="${l[0]} ${l[1]} ${l[2]}" rpy="0 0 0"/>
   </xacro:HDL-32E>
-  <xacro:cobot_v2_gazebo sim_drive="$(arg sim_drive)"/>
+  <!-- Front depth camera (RealSense D435). camera_depth_optical_frame: z forward, x right, y down. -->
+  <xacro:property name="c" value="${g['depth_camera_xyz']}"/>
+  <joint name="camera_joint" type="fixed">
+    <origin xyz="${c[0]} ${c[1]} ${c[2]}" rpy="0 0 0"/>
+    <parent link="base_link"/>
+    <child link="camera_link"/>
+  </joint>
+  <link name="camera_link">
+    <inertial>
+      <mass value="0.07"/>
+      <origin xyz="0 0 0"/>
+      <inertia ixx="1e-5" ixy="0" ixz="0" iyy="1e-5" iyz="0" izz="1e-5"/>
+    </inertial>
+    <visual>
+      <origin xyz="-0.0125 0 0"/>
+      <geometry><box size="0.025 0.09 0.025"/></geometry>
+      <material name="body_grey"/>
+    </visual>
+  </link>
+  <joint name="camera_depth_optical_joint" type="fixed">
+    <origin xyz="0 0 0" rpy="${-pi / 2} 0 ${-pi / 2}"/>
+    <parent link="camera_link"/>
+    <child link="camera_depth_optical_frame"/>
+  </joint>
+  <link name="camera_depth_optical_frame"/>
+  <xacro:cobot_v2_gazebo sim_drive="$(arg sim_drive)" depth_camera="$(arg depth_camera)"/>
 </robot>

Commit message: Add an IMU and fuse it with wheel odometry in a robot_localization EKF
- cobot_v2 gets an IMU link (mount in geometry.yaml: imu_xyz, imu_rpy; placeholder inside the lower
  body) and, in Gazebo, a 200 Hz IMU sensor on /imu/data with a typical MEMS gyro noise.
- base.launch (shared by the real robot and the simulation): kinematics_node publishes the wheel
  odometry on /wheel/odom only; ekf_odom (robot_localization EKF, config/ekf.yaml) fuses its body
  velocities with the IMU yaw rate and is the only publisher of /odom and TF odom -> base_footprint.
  ekf:=false keeps the previous wheel-odometry-only setup (also an argument of cobot_v2.launch).
- The Docker image installs robot_localization.

In sim_drive:=physics, where the wheels slip, the EKF keeps the heading that wheel odometry loses.

Co-Authored-By: Claude Opus 5.5 <noreply@anthropic.com>

File: wonik_cobot_v2_description/urdf/wonik_cobot_v2.gazebo.xacro (robot description, xacro)
@@ -95,4 +95,23 @@
       </gazebo>
     </xacro:if>
+    <!-- IMU: /imu/data (frame imu_link) at 200 Hz. The noise is a typical MEMS gyro (0.005 rad/s) and
+         also sets the message covariances (noise^2). No bias: robot_localization does not estimate one,
+         so a real gyro needs its bias removed by the driver (e.g. calibrated at standstill). -->
+    <gazebo reference="imu_link">
+      <sensor name="imu_sensor" type="imu">
+        <always_on>true</always_on>
+        <update_rate>200</update_rate>
+        <plugin name="imu_plugin" filename="libgazebo_ros_imu_sensor.so">
+          <topicName>imu/data</topicName>
+          <bodyName>imu_link</bodyName>
+          <frameName>imu_link</frameName>
+          <updateRateHZ>200.0</updateRateHZ>
+          <gaussianNoise>0.005</gaussianNoise>
+          <xyzOffset>0 0 0</xyzOffset>
+          <rpyOffset>0 0 0</rpyOffset>
+          <initialOrientationAsReference>false</initialOrientationAsReference>
+        </plugin>
+      </sensor>
+    </gazebo>
     <gazebo>
       <!-- Steer joints: position, drive joints: velocity (as on the real drive units). -->

File: wonik_cobot_v2_description/urdf/wonik_cobot_v2.urdf.xacro (robot description, xacro)
@@ -170,4 +170,19 @@
   </joint>
   <link name="camera_depth_optical_frame"/>
+  <!-- IMU: /imu/data in frame imu_link -->
+  <xacro:property name="i" value="${g['imu_xyz']}"/>
+  <xacro:property name="ir" value="${g['imu_rpy']}"/>
+  <joint name="imu_joint" type="fixed">
+    <origin xyz="${i[0]} ${i[1]} ${i[2]}" rpy="${ir[0]} ${ir[1]} ${ir[2]}"/>
+    <parent link="base_link"/>
+    <child link="imu_link"/>
+  </joint>
+  <link name="imu_link">
+    <inertial>
+      <mass value="0.01"/>
+      <origin xyz="0 0 0"/>
+      <inertia ixx="1e-6" ixy="0" ixz="0" iyy="1e-6" iyz="0" izz="1e-6"/>
+    </inertial>
+  </link>
   <xacro:cobot_v2_gazebo sim_drive="$(arg sim_drive)" depth_camera="$(arg depth_camera)"/>
 </robot>
