Commit message: cobot_v2 drive unit spec (WDS150): steering range, wheel speed limit
Wonik sent the drive unit drawing (WDS150, WDS-150-C260909); the same part
(WDS-LS48-400A-200A-FX1-Z1) is in cobot_v2_asm.stp. Wheel 150 x 55 mm,
steering +-140 deg at up to 2.56 rad/s, drive gear ratio left open on the
drawing (20 / 34 / 68 -> 1.18 / 0.69 / 0.35 m/s).
- geometry.yaml: wheel 0.150 x 0.055, steer_limit_deg 140, steer_max_vel;
  the URDF steer joints are revolute with these limits (were continuous)
- qd_kinematics: steer_limit. Steer commands took the shortest way round,
  which can cross +-180 deg (e.g. +130 -> -60 deg via 180); with a limited
  range they now move through the range. The node refuses a hysteresis band
  wider than the range.
- qd_kinematics: max_wheel_speed. A command that needs a faster wheel has all
  wheel speeds scaled by the same factor (same path, lower speed). cobot_v2:
  1.1775 m/s, assuming i = 20 until Wonik chooses the ratio.
- two unit tests (both fail on the previous controller); docs/safety.md: the
  steering encoder is incremental, so the driver must home it first
28 unit tests pass; cobot_v2 U route in Gazebo: no faults, steering within
[-1.5, 56.6] deg, cross-track max 3.9 cm.

Co-Authored-By: Claude Opus 5.5 <noreply@anthropic.com>

File: wonik_cobot_description/urdf/cobot_v2.urdf.xacro (robot description, xacro)
@@ -44,11 +44,13 @@
     </collision>
   </link>
-  <!-- QD unit: steer (continuous, position interface) + drive (continuous, velocity interface).
-       Steer frame sits on the steer axis at wheel-centre height; x = rolling direction at angle 0. -->
+  <!-- QD unit: steer (revolute within +-steer_limit_deg, position interface) + drive (continuous, velocity
+       interface). Steer frame sits on the steer axis at wheel-centre height; x = rolling direction at angle 0. -->
+  <xacro:property name="steer_limit" value="${g['steer_limit_deg'] * pi / 180.0}"/>
   <xacro:macro name="qd_unit" params="name x y">
-    <joint name="${name}_steer_joint" type="continuous">
+    <joint name="${name}_steer_joint" type="revolute">
       <origin xyz="${x} ${y} ${wheel_r}" rpy="0 0 0"/>
       <axis xyz="0 0 1"/>
       <dynamics damping="1.0"/>
+      <limit lower="${-steer_limit}" upper="${steer_limit}" effort="1000.0" velocity="${g['steer_max_vel']}"/>
       <parent link="base_link"/>
       <child link="${name}_steer_link"/>

Commit message: cobot_v2 drive unit spec (WDS150): steering range, wheel speed limit
Humble port of 21fe85e (main). Wonik sent the drive unit drawing (WDS150,
WDS-150-C260909); the same part (WDS-LS48-400A-200A-FX1-Z1) is in
cobot_v2_asm.stp. Wheel 150 x 55 mm, steering +-140 deg at up to 2.56 rad/s,
drive gear ratio i = 20 (1.18 m/s; the drawing also offers 34 / 68 ->
0.69 / 0.35 m/s).
- geometry.yaml: wheel 0.150 x 0.055, steer_limit_deg 140, steer_max_vel;
  the URDF steer joints are revolute with these limits (were continuous), and
  the steer position command interfaces in the ros2_control tags carry the
  same min/max
- base.launch.py passes steer_limit_deg from geometry.yaml to kinematics_node
  (the launch copies only listed geometry keys)
- qd_kinematics: steer_limit. Steer commands took the shortest way round,
  which can cross +-180 deg (e.g. +130 -> -60 deg via 180); with a limited
  range they now move through the range. The node refuses a hysteresis band
  wider than the range.
- qd_kinematics: max_wheel_speed. A command that needs a faster wheel has all
  wheel speeds scaled by the same factor (same path, lower speed). cobot_v2:
  1.1775 m/s, gear ratio i = 20.
- two unit tests (both fail on the previous controller); docs/safety.md: the
  steering encoder is incremental, so the driver must home it first
28 unit tests pass; cobot_v2 U route in Gazebo (headless): no faults,
steering within [-0.6, 56.6] deg, cross-track max 4.6 cm.

Co-Authored-By: Claude Opus 5.5 <noreply@anthropic.com>

File: wonik_cobot_description/urdf/cobot_v2.urdf.xacro (robot description, xacro)
@@ -43,11 +43,13 @@
     </collision>
   </link>
-  <!-- QD unit: steer (continuous, position interface) + drive (continuous, velocity interface).
-       Steer frame sits on the steer axis at wheel-centre height; x = rolling direction at angle 0. -->
+  <!-- QD unit: steer (revolute within +-steer_limit_deg, position interface) + drive (continuous, velocity
+       interface). Steer frame sits on the steer axis at wheel-centre height; x = rolling direction at angle 0. -->
+  <xacro:property name="steer_limit" value="${g['steer_limit_deg'] * pi / 180.0}"/>
   <xacro:macro name="qd_unit" params="name x y">
-    <joint name="${name}_steer_joint" type="continuous">
+    <joint name="${name}_steer_joint" type="revolute">
       <origin xyz="${x} ${y} ${wheel_r}" rpy="0 0 0"/>
       <axis xyz="0 0 1"/>
       <dynamics damping="1.0"/>
+      <limit lower="${-steer_limit}" upper="${steer_limit}" effort="1000.0" velocity="${g['steer_max_vel']}"/>
       <parent link="base_link"/>
       <child link="${name}_steer_link"/>
@@ -195,5 +197,8 @@
       <xacro:if value="${i &lt; len(g['module_names'])}">
         <joint name="${g['steer_joints'][i]}">
-          <command_interface name="position"/>
+          <command_interface name="position">
+            <param name="min">${-steer_limit}</param>
+            <param name="max">${steer_limit}</param>
+          </command_interface>
           <state_interface name="position"><param name="initial_value">0.0</param></state_interface>
           <state_interface name="velocity"/>
